File: CurrentBoard/CurrentSource.sch (KiCad schematic (older format))
At the start: 2 parts, among them U1 LMV358

Commit message: 17-8-19-2017
Parts:
- removed U1: LMV358, symbol LMV358
- removed U?: INA180, symbol INA180
- added C? (x2): C, symbol C
- added R?: 1.6, Resistors_SMD:R_2512_HandSoldering, symbol R
- added R? (x4): R, symbol R
- added U?: TLV3201AQDCKRQ1, kicad-libraries-master:SC70-5, symbol TLV3201AQDCKRQ1
- added U?: INA180, TO_SOT_Packages_SMD:SOT-23-5_HandSoldering, symbol INA180
Connections:
- net labels added: +5V, GND, shunt_in, shunt_out, square_wave
- wire segments 0 -> 32
Other:
- note added: "SHUNT & AMP\n"
- note added: "SQUARE WAVE GENERATOR\n"

Commit message: 17-8-20-2329
Parts:
- removed R?: R, symbol R
- added C? (x3): C, symbol C
- added R? (x3): R, symbol R
- added RV?: 1M, symbol POT
- added U?: SN74LVC1G175, symbol SN74LVC1G175
- added U? (x2): ADA4891, SMD_Packages:SOIC-14_N, symbol ADA4891
- added U? (x2): ADA4891, symbol ADA4891
- C?: value C -> 100p
Connections:
- net +5V: now also C?.1, C?.1, C?.1, R?.1, U?.4 (V+), U?.5 (VCC)
- net GND: now also C?.2, C?.2, C?.2, U?.11 (V-), U?.2 (GND)
- net at C?.1, U?.4 (IN-): now also RV?.2
- net shunt_out: no longer names the net of U?.1 (OUT)
- net shunt_out: now also U?.2 (-)
- net square_wave: no longer names the net of R?.1, U?.1 (OUT)
- net square_wave: now also RV?.3, U?.1 (CLK)
- new net: R?.2, U?.3 (D)
- new net: R?.1, U?.1, U?.6 (~CLR)
- new net: R?.1, R?.2, U?.3 (+)
- new net DAC_IN: R?.2
Other:
- note added: "CONTROL COMPARITOR\n"
- note added: "DFF MOSFET CONTROLLER\n"

Commit message: 17-8-24-0030
Parts:
- added C? (x3): C, symbol C
- added R? (x3): R, symbol R
- added U?: MCP4725, symbol MCP4725
- added U?: UCC27517A, symbol UCC27517A
Connections:
- net +5V: now also C?.2, C?.2, C?.2, R?.1, R?.1, U?.1 (VDD), U?.3 (Vdd)
- net GND: now also C?.1, C?.1, C?.1, U?.2 (GND), U?.2 (Vss), U?.4 (IN-), U?.6 (A0)
- net at U?.4 (Q): now also U?.3 (IN+)
- net DAC_IN renamed SMCS_REF
- new net: R?.1, U?.5 (OUT)
- new net DAC_OUT: U?.1 (Vout)
- new net DAC_SCL: R?.2, U?.5 (SCL)
- new net DAC_SDA: R?.2, U?.4 (SDA)
- new net MOSFET_DRIVER: R?.2
Other:
- note added: "MOSFET DRIVER\n\n"
- note added: "REFERENCE DAC\n\n"
- moved on the sheet: U?B, U?C, U?D

Commit message: 17-8-26-2228
Parts:
- added C? (x2): C, symbol C
- added Con? (x6): 1x1Connector, symbol 1x1Connector
- added R? (x4): R, symbol R
- added RV?: 1M, symbol POT
- added U?: PIC16F15325, SMD_Packages:SOIC-14_N, symbol PIC16F15325
Connections:
- net +5V: now also C?.2, R?.1, R?.1, R?.2, RV?.3, U?.1 (Vdd)
- net DAC_SCL: now also R?.2, U?.10 (RC0)
- net DAC_SDA: now also R?.1, U?.11 (RA2)
- net GND: now also C?.1, C?.2, RV?.1, U?.14 (Vss)
- net SMCS_REF: now also Con?.~
- net DAC_OUT: no longer names the net of U?.1 (Vout)
- net DAC_OUT: now also Con?.~
- new net: Con?.~, U?.12 (RA1/ICSPCLK)
- new net: Con?.~, U?.13 (RA0/ICSPDAT)
- new net: Con?.~, R?.2, U?.4 (RA3/~MCLR~/Vpp)
- new net: C?.1, R?.1, R?.2
- new net: Con?.~, RV?.2
Other:
- note added: "MICROCONTROLLER\n"
- note added: "REFERENCE\n\n"
- note removed: "REFERENCE DAC\n\n"
- moved on the sheet: U?B, U?C, U?D

Commit message: 17-8-28-2311
Parts:
- added C? (x2): C, symbol C
- added Con? (x6): 1x1Connector, symbol 1x1Connector
- added J?: USB_OTG, symbol USB_OTG
- added R? (x4): R, symbol R
- added U?: MCP2221, symbol MCP2221
- gave numbers to parts that had none: 39
Connections:
- net +5V: now also C?.1, R?.1, R?.1, R?.2, U?.1 (Vdd)
- net GND: now also C?.1, C?.2, J?.5 (GND), J?.6 (Shield), R?.1, U?.14 (Vss)
- net at U3.8 (RC2): now also Con?.~
- net at U3.9 (RC1): now also Con?.~
- new net: J?.1 (VBUS), R?.2
- new net: J?.2 (D-), U?.12 (D-)
- new net: J?.3 (D+), U?.13 (D+)
- new net: Con?.~, R?.1, U?.10 (SCL)
- new net: C?.2, U?.11 (Vusb)
- new net: R?.2, U?.4 (~RST)
- new net: Con?.~, U?.5 (URx)
- new net: Con?.~, U?.6 (UTx)
- new net: Con?.~, R?.2, U?.9 (SDA)
Other:
- note added: "USB -> UART Bridge\n"
